File: dac_controller_3x2.kicad_pcb (KiCad board)
At the start: 2 copper layers, 70.5 x 41.9 mm, 1 part

Commit message: Initial layout.
Parts:
- added C1: 10uF, dac_controller_3x2:SM1210, B.Cu at (102.2, 96.5)
- added C2: 0.1uF, dac_controller_3x2:SM1210, B.Cu at (130.2, 81.3)
- added C3: 10uF, dac_controller_3x2:SM1210, B.Cu at (111.8, 85.1)
- added C4: 0.1uF, dac_controller_3x2:SM1210, B.Cu at (118.1, 85.1)
- added C5: 10uF, dac_controller_3x2:SM1210, B.Cu at (111.8, 80.0)
- added C6: 0.1uF, dac_controller_3x2:SM1210, B.Cu at (118.1, 80.0)
- added D1: AD5754R, dac_controller_3x2:TSSOP_EP_24, B.Cu at (130.2, 88.9)
- added P1: BNC_DOUBLE_RA, dac_controller_3x2:BNC_DOUBLE, F.Cu at (150.5, 102.2)
- added P2: BNC_DOUBLE_RA, dac_controller_3x2:BNC_DOUBLE, F.Cu at (150.5, 75.6)
- added REG1: CONV_DC_DC_-12V_12V_1W, dac_controller_3x2:DC_DC_CONV_RSO, F.Cu at (107.3, 88.9)
Connections:
- MDB1 pad 10: (no net) -> /CS
- MDB1 pad 11: (no net) -> /MOSI
- MDB1 pad 12: (no net) -> /MISO
- MDB1 pad 13: (no net) -> /SCK
- MDB1 pad 3: (no net) -> /LDAC
- MDB1 pad 4: (no net) -> /CLR
- MDB1 pad GND: (no net) -> GND
- MDB1 pad VDD: (no net) -> VDD
- MDB1 pad VEE: (no net) -> VEE
Routing:
- net GND: track 0.00 -> 169.2 mm, vias 0 -> 1
- net /CS: track 0.00 -> 61.2 mm
- net VEE: track 0.00 -> 52.1 mm, vias 0 -> 1
- net VSSA: track 0.00 -> 46.7 mm, vias 0 -> 1
- net /CLR: track 0.00 -> 43.9 mm
- net VDDA: track 0.00 -> 42.7 mm, vias 0 -> 1
- net /LDAC: track 0.00 -> 41.6 mm, vias 0 -> 1
- net VDD: track 0.00 -> 35.7 mm
- net /MOSI: track 0.00 -> 28.0 mm
- net /MISO: track 0.00 -> 18.5 mm
- net /SCK: track 0.00 -> 17.9 mm
- net /dac_3x2/VoutA: track 0.00 -> 16.7 mm
- net /dac_3x2/VoutC: track 0.00 -> 16.6 mm
- net /dac_3x2/VoutB: track 0.00 -> 15.2 mm
- net /dac_3x2/VoutD: track 0.00 -> 14.9 mm
- added copper zone on B.Cu, net GND
- added copper zone on F.Cu, net GND
Other:
- net class LEDPOWER: clearance 0.254 -> 0.1016; trace_width 0.6096 -> 0.4064
- net class POWER: clearance 0.254 -> 0.1016; trace_width 0.8128 -> 0.4064
- net class SUPERPOWER: clearance 0.254 -> 0.1016; trace_width 1.2192 -> 0.6096
- board text added: "Janelia Modular Device dac_controller part_number: 1281 09/2018 ver 1.0 3x2"
- board text removed: "Janelia Modular Device dac_controller part_number: 1001 02/2017 ver 1.0 3x2"

Commit message: Finished v1.0.
Connections:
- net /dac_3x2/VoutA renamed /dac_3x2/DAC_0
- net /dac_3x2/VoutB renamed /dac_3x2/DAC_1
- net /dac_3x2/VoutC renamed /dac_3x2/DAC_2
- net /dac_3x2/VoutD renamed /dac_3x2/DAC_3
Other:
- board text added: "+/-12VDC"
